File: hardware/pico-poe/pico-poe.kicad_pcb (KiCad board)
At the start: 4 copper layers, 68.6 x 21 mm, 76 parts, among them J1 PinSocket-20, J2 PinSocket-20, J3 RJHSE5385, U1 LM5160A, U2 TPS2378, U3 TLP290, U4 AP63205WU, U5 LAN8720A

Commit message: touchup + purchase
Routing:
- net +3.3V_ISO: track 103.0 -> 60.7 mm, vias 1 -> 2
Other:
- board text added: "12V 2A"
- board text added: "2026 PICO-POE"
- board text added: "2026 RM1N"
- board text added: "LAN8720A"
- board text added: "PICO-POE REVA"
- board text added: "RM1N"
- board text added: "©"
