File: hardware/c0-dev/c0-dev.kicad_pcb (KiCad board)
At the start: 2 copper layers, 446 parts, among them J101 2913730000, J102 2913710000, J103 2913730000, J104 2913730000, J105 2913730000, J106 2913710000, J107 2913730000, J108 2913730000, J109 2913730000, J111 2913730000, J112 2913730000, J113 2913730000, J114 2913730000, J201 RJ45_LED_Shielded, J401 TAG_CONNECT, J402 PinHeader_2.54mm, Q1001 BSS138P, Q1002 BSS138P, Q1003 BSS138P, Q1004 BSS138P, Q1005 BSS138P, Q1006 BSS138P, Q1007 BSS138P, Q1008 BSS138P, Q1009 BSS138P, Q701 BSS138P, Q702 BSS138P, U1001 TCA9555PWR, U1002 TPS4H000A-Q1, U1003 TPS4H000A-Q1, U1101 LM5160A, U1102 LM317L, U1201 ER_OLEDM0.91_1x-I2C, U1301 TPS4H000A-Q1, U201 LAN8720A, U301 AP63203WU, U302 TPS2378, U303 TPS54360DDA, U304 TLP175A, U401 TCA9555PWR, U402 W25Q128JVP, U403 TPS3820-33DBV, U404 RP2350A, U501 B0505S-1WR3, U502 ISO1540, U503 ISO1540, U504 AMS1117-3.3, U505 TMP117xxDRV, U506 ADS1015IDGS, U507 ADS1015IDGS, U601 ADS1015IDGS, U602 ADS1015IDGS, U603 ADS1015IDGS, U604 ADS1015IDGS, U701 B0505S-1WR3, U702 ISO6741, U703 ISO6741, U704 ADS1220xPW, U705 ADS1220xPW, U801 B0505S-1WR3, U802 ISO1044BD, U803 TLP175A, U901 ISO1212, U902 ISO1212, U903 ISO1212, U904 ISO1212, Y401 ABM8-272-T3 (12Mhz)

Commit message: added LEDs
Parts:
- removed J106: 2913710000, conduit:2913710000
- removed J114: 2913730000, conduit:2913730000
- added C526: 0.1uF, Capacitor_SMD:C_0402_1005Metric, F.Cu at (339.5, 117.9)
- added J110: 2913730000, conduit:2913730000, F.Cu at (187.8, 103.1)
- added R524: 1M, Resistor_SMD:R_0402_1005Metric, F.Cu at (336.8, 125.8)
- added R525: 1M, Resistor_SMD:R_0402_1005Metric, F.Cu at (336.8, 127.8)
- added R526: 1M, Resistor_SMD:R_0402_1005Metric, F.Cu at (336.8, 129.8)
- added U508: ADS1015IDGS, Package_SO:TSSOP-10_3x3mm_P0.5mm, F.Cu at (344.6, 117.9)
- C509: value 1uF -> 0.1uF
- C511: value 0.1uF -> 1uF
- R508, R509, R510: value 2k -> 1k; footprint Resistor_SMD:R_1206_3216Metric -> Resistor_SMD:R_0402_1005Metric
- R516, R517, R518: value 1M -> 2k; footprint Resistor_SMD:R_0402_1005Metric -> Resistor_SMD:R_1206_3216Metric
- U504: value AMS1117-3.3 -> TMP117xxDRV; footprint Package_TO_SOT_SMD:SOT-223-3_TabPin2 -> Package_SON:WSON-6-1EP_2x2mm_P0.65mm_EP1x1.6mm
- U505: value TMP117xxDRV -> AMS1117-3.3; footprint Package_SON:WSON-6-1EP_2x2mm_P0.65mm_EP1x1.6mm -> Package_TO_SOT_SMD:SOT-223-3_TabPin2
- U506: value ADS1015IDGS -> TMP117xxDRV; footprint Package_SO:TSSOP-10_3x3mm_P0.5mm -> Package_SON:WSON-6-1EP_2x2mm_P0.65mm_EP1x1.6mm
- moved C801 351.5 mm to (391.2, 141.2)
- moved C802 351.5 mm to (391.2, 144.2)
- moved C803 351.5 mm to (391.2, 147.2)
- moved C804 351.5 mm to (398.9, 138.5)
- moved C805 351.5 mm to (391.2, 150.2)
- moved D801 351.5 mm to (397.5, 147.1)
- moved D802 351.5 mm to (399.9, 135.3)
- moved FB801 351.5 mm to (383.2, 150.5)
- moved R801 351.5 mm to (387.0, 147.3)
- moved R802 351.5 mm to (383.4, 147.8)
- moved R803 351.5 mm to (387.0, 149.3)
- moved U801 351.5 mm to (383.2, 136.1)
- moved U802 351.5 mm to (393.2, 136.5)
- moved U803 351.5 mm to (397.9, 142.3)
- moved C712 326.2 mm to (388.3, 48.4)
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Connections:
- C514 pad 1: Net-(D502B-K1A2) -> +3.3V
- C515 pad 2: Net-(D502A-K3A4) -> GND
- C516 pad 1: Net-(D502A-K3A4) -> Net-(D502B-K1A2)
- C516 pad 2: GND -> Net-(D502A-K3A4)
- C517 pad 1: Net-(D503B-K1A2) -> Net-(D502A-K3A4)
- C518 pad 2: Net-(D503A-K3A4) -> GND
- C519 pad 1: Net-(D503A-K3A4) -> Net-(D503B-K1A2)
- C519 pad 2: GND -> Net-(D503A-K3A4)
- C520 pad 1: Net-(D504B-K1A2) -> Net-(D503A-K3A4)
- C521 pad 2: Net-(D504A-K3A4) -> GND
- C522 pad 1: Net-(D504A-K3A4) -> Net-(D504B-K1A2)
- C522 pad 2: GND -> Net-(D504A-K3A4)
- C523 pad 1: Net-(D505B-K1A2) -> Net-(D504A-K3A4)
- C524 pad 2: Net-(D505A-K3A4) -> GND
- C525 pad 1: Net-(D505A-K3A4) -> Net-(D505B-K1A2)
- C525 pad 2: GND -> Net-(D505A-K3A4)
- J111 pad 1: /frontend_temp/TC0+ -> /frontend_bridge/B1_5V+
- J111 pad 2: /frontend_temp/TC0- -> /frontend_bridge/B1+
- J111 pad 3: /frontend_temp/TC1+ -> /frontend_bridge/B1-
- J111 pad 4: /frontend_temp/TC1- -> /frontend_bridge/B1_GND
- J112 pad 1: /frontend_temp/TC2+ -> /frontend_temp/TC0+
- J112 pad 2: /frontend_temp/TC2- -> /frontend_temp/TC0-
- J112 pad 3: /frontend_temp/TC3+ -> /frontend_temp/TC1+
- J112 pad 4: /frontend_temp/TC3- -> /frontend_temp/TC1-
- J113 pad 1: /frontend_bridge/B0_5V+ -> /frontend_temp/TC2+
- J113 pad 2: /frontend_bridge/B0+ -> /frontend_temp/TC2-
- J113 pad 3: /frontend_bridge/B0- -> /frontend_temp/TC3+
- J113 pad 4: /frontend_bridge/B0_GND -> /frontend_temp/TC3-
- R1308 pad 1: /Power Output/~{FLT} -> /FAULT_PWR
- R501 pad 1: /MCU/I2C0.SCL -> /frontend_temp/SDA_400k
- R502 pad 1: /frontend_temp/SDA_400k -> /frontend_temp/SCL_400k
- R503 pad 1: /MCU/I2C0.SDA -> +3.3V
- R503 pad 2: +3.3V -> Net-(U504-ADD0)
- R504 pad 1: /frontend_temp/SCL_400k -> /frontend_temp/SDA_400k
- R505 pad 1: GND -> /frontend_temp/SCL_400k
- R505 pad 2: Net-(U506-ADDR) -> +3.3V
- R506 pad 2: Net-(U505-ADD0) -> Net-(U506-ADD0)
- R507 pad 1: +3.3V -> /MCU/I2C0.SCL
- R507 pad 2: Net-(U507-ADDR) -> +3.3V
- R508 pad 1: /frontend_temp/TC0- -> /MCU/I2C0.SDA
- R508 pad 2: Net-(D502B-K1A2) -> +3.3V
- R509 pad 1: /frontend_temp/TC0+ -> GND
- R509 pad 2: Net-(D502A-K3A4) -> Net-(U507-ADDR)
- R510 pad 1: /frontend_temp/TC1- -> +3.3V
- R510 pad 2: Net-(D503B-K1A2) -> Net-(U508-ADDR)
- R511 pad 1: /frontend_temp/TC1+ -> /frontend_temp/TC0-
- R511 pad 2: Net-(D503A-K3A4) -> Net-(D502B-K1A2)
- R512 pad 1: /frontend_temp/TC2- -> /frontend_temp/TC0+
- R512 pad 2: Net-(D504B-K1A2) -> Net-(D502A-K3A4)
- R513 pad 1: /frontend_temp/TC2+ -> /frontend_temp/TC1-
- R513 pad 2: Net-(D504A-K3A4) -> Net-(D503B-K1A2)
- R514 pad 1: /frontend_temp/TC3- -> /frontend_temp/TC1+
- R514 pad 2: Net-(D505B-K1A2) -> Net-(D503A-K3A4)
- R515 pad 1: /frontend_temp/TC3+ -> /frontend_temp/TC2-
- R515 pad 2: Net-(D505A-K3A4) -> Net-(D504B-K1A2)
- R516 pad 1: /frontend_temp/TC0- -> /frontend_temp/TC2+
- R516 pad 2: +3.3V -> Net-(D504A-K3A4)
- R517 pad 1: GND -> /frontend_temp/TC3-
- R517 pad 2: /frontend_temp/TC0+ -> Net-(D505B-K1A2)
- R518 pad 1: /frontend_temp/TC1- -> /frontend_temp/TC3+
- R518 pad 2: +3.3V -> Net-(D505A-K3A4)
- R519 pad 1: GND -> /frontend_temp/TC0-
- R519 pad 2: /frontend_temp/TC1+ -> +3.3V
- R520 pad 1: /frontend_temp/TC2- -> GND
- R520 pad 2: +3.3V -> /frontend_temp/TC0+
- R521 pad 1: GND -> /frontend_temp/TC1-
- R521 pad 2: /frontend_temp/TC2+ -> +3.3V
- R522 pad 1: /frontend_temp/TC3- -> GND
- R522 pad 2: +3.3V -> /frontend_temp/TC1+
- R523 pad 1: GND -> /frontend_temp/TC2-
- R523 pad 2: /frontend_temp/TC3+ -> +3.3V
- U1301 pad 5: /Power Output/~{FLT} -> /FAULT_PWR
- U1301 pad 6: /Power Output/~{FLT} -> /FAULT_PWR
- U1301 pad 7: /Power Output/~{FLT} -> /FAULT_PWR
- U1301 pad 8: /Power Output/~{FLT} -> /FAULT_PWR
- U401 pad 8: /FAULT_420 -> /FAULT_PWR
- U504 pad 1: GND -> /frontend_temp/SCL_400k
- U504 pad 2: +3.3V -> GND
- U504 pad 3: /frontend_temp/+5V_ISO -> unconnected-(U504-ALERT-Pad3)
- U505 pad 1: /frontend_temp/SCL_400k -> GND
- U505 pad 2: GND -> +3.3V
- U505 pad 3: unconnected-(U505-ALERT-Pad3) -> /frontend_temp/+5V_ISO
- U506 pad 1: Net-(U506-ADDR) -> /frontend_temp/SCL_400k
- U506 pad 2: unconnected-(U506-ALERT/RDY-Pad2) -> GND
- U506 pad 3: GND -> unconnected-(U506-ALERT-Pad3)
- U506 pad 4: Net-(D502B-K1A2) -> Net-(U506-ADD0)
- U506 pad 5: Net-(D502A-K3A4) -> +3.3V
- U506 pad 6: Net-(D503B-K1A2) -> /frontend_temp/SDA_400k
- U506 pad 7: Net-(D503A-K3A4) -> /frontend_temp/TC0-
- U507 pad 4: Net-(D504B-K1A2) -> Net-(D502B-K1A2)
- U507 pad 5: Net-(D504A-K3A4) -> Net-(D502A-K3A4)
- U507 pad 6: Net-(D505B-K1A2) -> Net-(D503B-K1A2)
- U507 pad 7: Net-(D505A-K3A4) -> Net-(D503A-K3A4)
Other:
- board outline added: 160 x 100 mm

Commit message: rgb's and 70x160mm
Parts:
- added H101: MountingHole, MountingHole:MountingHole_3.2mm_M3_DIN965_Pad_TopBottom, F.Cu at (64.0, 126.0)
- added H102: MountingHole, MountingHole:MountingHole_3.2mm_M3_DIN965_Pad_TopBottom, F.Cu at (130.2, 125.0)
- added H103: MountingHole, MountingHole:MountingHole_3.2mm_M3_DIN965_Pad_TopBottom, F.Cu at (64.0, 66.0)
- added H104: MountingHole, MountingHole:MountingHole_3.2mm_M3_DIN965_Pad_TopBottom, F.Cu at (216.0, 126.0)
- added H105: MountingHole, MountingHole:MountingHole_3.2mm_M3_DIN965_Pad_TopBottom, F.Cu at (136.0, 66.0)
- added H106: MountingHole, MountingHole:MountingHole_3.2mm_M3_DIN965_Pad_TopBottom, F.Cu at (216.0, 66.0)
- moved L1101 42.9 mm to (86.0, 71.0)
- moved J201 38.7 mm to (75.5, 75.5)
- moved J101 18.2 mm to (92.0, 126.0)
- moved J102 18.2 mm to (92.0, 103.0)
- moved U1201 11.1 mm to (70.2, 91.5), turned to 0 degrees
- moved J103 8.80 mm to (158.2, 103.0)
- moved J104 8.80 mm to (138.0, 126.0)
- moved J105 8.80 mm to (138.0, 102.5)
- moved J109 8.80 mm to (158.0, 126.5)
- moved J110 8.80 mm to (179.0, 103.1)
- moved J111 8.80 mm to (179.0, 126.5)
- moved J107 8.80 mm to (115.0, 125.5)
- moved J108 8.80 mm to (115.0, 102.5)
- moved J112 6.00 mm to (201.8, 103.5)
- moved J113 6.00 mm to (201.8, 126.5)
Other:
- board size 160 x 100 mm -> 160 x 70 mm

Commit message: started PCB
Parts:
- removed C1116: 4.7nF, Capacitor_SMD:C_0402_1005Metric
- removed C307, C309: 1uF, Capacitor_SMD:C_1206_3216Metric
- removed J113: 2913730000, conduit:2913730000
- removed R1109: 51k, Resistor_SMD:R_0402_1005Metric
- removed R219: 33R, Resistor_SMD:R_0402_1005Metric
- added C101: 1nF, Capacitor_SMD:C_1206_3216Metric, F.Cu at (333.4, 121.7)
- added C102: 1nF, Capacitor_SMD:C_1206_3216Metric, F.Cu at (333.4, 125.1)
- added C103: 1nF, Capacitor_SMD:C_1206_3216Metric, F.Cu at (333.4, 128.4)
- added C1202: 10uF, Capacitor_SMD:C_0805_2012Metric, F.Cu at (339.6, 96.1)
- added D1201: WS2812B, LED_SMD:LED_WS2812B_PLCC4_5.0x5.0mm_P3.2mm, F.Cu at (333.3, 94.9)
- added D1202: WS2812B, LED_SMD:LED_WS2812B_PLCC4_5.0x5.0mm_P3.2mm, F.Cu at (333.3, 101.5)
- added J106: 2913730000, conduit:2913730000, F.Cu at (105.0, 104.0)
- added R101: 2M, Resistor_SMD:R_1206_3216Metric, F.Cu at (339.0, 121.7)
- added R102: 2M, Resistor_SMD:R_1206_3216Metric, F.Cu at (339.0, 125.0)
- added R103: 2M, Resistor_SMD:R_1206_3216Metric, F.Cu at (339.0, 128.3)
- added R423: 1k, Resistor_SMD:R_0402_1005Metric, F.Cu at (255.0, 133.2)
- added R527: 0, Resistor_SMD:R_0402_1005Metric, F.Cu at (204.0, 74.0)
- added R719: 0, Resistor_SMD:R_0402_1005Metric, F.Cu at (312.4, 60.4)
- C1104, C1108, C1109, C1110, C1111, C208, C209, C210, C211, C313, D1101, D1102, D303, D304, R1103, R214, R215, R216, R307, R312, U1101, U304: moved to B.Cu
- C1113: value 1nF -> 10uF; footprint Capacitor_SMD:C_1206_3216Metric -> Capacitor_SMD:C_1210_3225Metric; moved to B.Cu
- C1114: value 10uF -> 10nF; footprint Capacitor_SMD:C_1210_3225Metric -> Capacitor_SMD:C_0402_1005Metric; moved to B.Cu
- C1115: value 10nF -> 4.7nF; moved to B.Cu
- C414: value 0.1u -> 15p
- C416: value 15p -> 0.1u
- H101, H102, H103, H104, H105, H106: value MountingHole -> M3; footprint MountingHole:MountingHole_3.2mm_M3_DIN965_Pad_TopBottom -> MountingHole:MountingHole_3.5mm_Pad_TopBottom
- J102: value 2913710000 -> 2913730000; footprint conduit:2913710000 -> conduit:2913730000
- R1106: value 2M -> 27k; footprint Resistor_SMD:R_1206_3216Metric -> Resistor_SMD:R_0402_1005Metric; moved to B.Cu
- R1107: value 27k -> 2.4k; moved to B.Cu
- R1108: value 2.4k -> 51k; moved to B.Cu
- R213: value 2M -> 75R; footprint Resistor_SMD:R_1206_3216Metric -> Resistor_SMD:R_0402_1005Metric; moved to B.Cu
- R217: value 75R -> 33R
- R409: value 1k -> DNP
- R410: value DNP -> 0
- R411: value 0 -> 27
- R413: value 27 -> 10k
- R414: value 1k -> 27
- R415: value 10k -> 1k
- R416: value 27 -> 1k
- R422: value 1k -> 0
- U403: value TPS3820-33DBV -> RP2350A; footprint Package_TO_SOT_SMD:SOT-23-5 -> Package_DFN_QFN:QFN-60-1EP_7x7mm_P0.4mm_EP3.4x3.4mm
- U404: value RP2350A -> TPS3820-33DBV; footprint Package_DFN_QFN:QFN-60-1EP_7x7mm_P0.4mm_EP3.4x3.4mm -> Package_TO_SOT_SMD:SOT-23-5
- moved C301 331.1 mm to (80.0, 96.0)
- moved C201 321.1 mm to (55.5, 95.0)
- moved C202 321.1 mm to (55.5, 97.0)
- moved C203 321.1 mm to (55.5, 99.0)
- moved C204 321.1 mm to (55.5, 100.9)
- moved C205 321.1 mm to (55.5, 102.9)
- moved C206 321.1 mm to (55.5, 104.9)
- moved C207 321.1 mm to (55.5, 106.8)
- moved R207 321.1 mm to (49.7, 95.0)
- moved R208 321.1 mm to (49.7, 97.0)
- moved R209 321.1 mm to (49.7, 99.0)
- moved R210 321.1 mm to (49.7, 101.0)
- moved R211 321.1 mm to (49.7, 103.0)
- moved R212 321.1 mm to (49.7, 105.0)
- moved FB201 321.1 mm to (46.8, 95.0)
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Connections:
- C1112 pad 1: +24V -> /Power/FlyBuck/+24V_PRIM
- C1113 pad 1: GND -> /Power/FlyBuck/+24V_PRIM
- C1113 pad 2: Earth -> /Power/GND_ISO
- C1114 pad 1: +24V -> /Power/FlyBuck/A
- C1114 pad 2: /Power/GND_ISO -> /Power/FlyBuck/FB
- C1115 pad 2: /Power/FlyBuck/FB -> /Power/GND_ISO
- C414 pad 1: +3.3V -> GND
- C414 pad 2: GND -> Net-(U403-XIN)
- C415 pad 2: Net-(U404-XIN) -> Net-(C415-Pad2)
- C416 pad 1: GND -> +3.3V
- C416 pad 2: Net-(C416-Pad2) -> GND
- C504 pad 2: GND -> /frontend_temp/GND
- C505 pad 1: +3.3V -> /frontend_temp/+3.3V
- C505 pad 2: GND -> /frontend_temp/GND
- C506 pad 2: GND -> /frontend_temp/GND
- C507 pad 1: +3.3V -> /frontend_temp/+3.3V
- C507 pad 2: GND -> /frontend_temp/GND
- C508 pad 1: +3.3V -> /frontend_temp/+3.3V
- C508 pad 2: GND -> /frontend_temp/GND
- C509 pad 1: +3.3V -> /frontend_temp/+3.3V
- C509 pad 2: GND -> /frontend_temp/GND
- C510 pad 1: +3.3V -> /frontend_temp/+3.3V
- C510 pad 2: GND -> /frontend_temp/GND
- C511 pad 1: +3.3V -> /frontend_temp/+3.3V
- C511 pad 2: GND -> /frontend_temp/GND
- C512 pad 1: +3.3V -> /frontend_temp/+3.3V
- C512 pad 2: GND -> /frontend_temp/GND
- C513 pad 1: +3.3V -> /frontend_temp/+3.3V
- C513 pad 2: GND -> /frontend_temp/GND
- C514 pad 1: +3.3V -> /frontend_temp/+3.3V
- C514 pad 2: GND -> /frontend_temp/GND
- C515 pad 2: GND -> /frontend_temp/GND
- C517 pad 2: GND -> /frontend_temp/GND
- C518 pad 2: GND -> /frontend_temp/GND
- C520 pad 2: GND -> /frontend_temp/GND
- C521 pad 2: GND -> /frontend_temp/GND
- C523 pad 2: GND -> /frontend_temp/GND
- C524 pad 2: GND -> /frontend_temp/GND
- C526 pad 2: GND -> /frontend_temp/GND
- C701 pad 1: +5V_ISO -> +5V
- C701 pad 2: GND_ISO -> GND
- C704 pad 2: GND -> /frontend_bridge/GND
- C705 pad 2: GND -> /frontend_bridge/GND
- C706 pad 2: GND -> /frontend_bridge/GND
- C707 pad 2: GND -> /frontend_bridge/GND
- C708 pad 2: GND -> /frontend_bridge/GND
- C709 pad 2: GND -> /frontend_bridge/GND
- C710 pad 2: GND -> /frontend_bridge/GND
- C711 pad 2: GND -> /frontend_bridge/GND
- C714 pad 2: GND -> /frontend_bridge/GND
- C716 pad 2: GND -> /frontend_bridge/GND
- C717 pad 2: GND -> /frontend_bridge/GND
- C719 pad 2: GND -> /frontend_bridge/GND
- C801 pad 1: +5V_ISO -> +5V
- C801 pad 2: GND_ISO -> GND
- C803 pad 2: GND -> /CAN/GND
- C804 pad 2: GND -> /CAN/GND
- C805 pad 2: GND -> /CAN/GND
- D502 pad 1: GND -> /frontend_temp/GND
- D502 pad 2: +3.3V -> /frontend_temp/+3.3V
- D502 pad 4: GND -> /frontend_temp/GND
- D502 pad 5: +3.3V -> /frontend_temp/+3.3V
- D503 pad 1: GND -> /frontend_temp/GND
- D503 pad 2: +3.3V -> /frontend_temp/+3.3V
- D503 pad 4: GND -> /frontend_temp/GND
- D503 pad 5: +3.3V -> /frontend_temp/+3.3V
- D504 pad 1: GND -> /frontend_temp/GND
- D504 pad 2: +3.3V -> /frontend_temp/+3.3V
- D504 pad 4: GND -> /frontend_temp/GND
- D504 pad 5: +3.3V -> /frontend_temp/+3.3V
- D505 pad 1: GND -> /frontend_temp/GND
- D505 pad 2: +3.3V -> /frontend_temp/+3.3V
- D505 pad 4: GND -> /frontend_temp/GND
- D505 pad 5: +3.3V -> /frontend_temp/+3.3V
- D506 pad 2: GND -> /frontend_temp/GND
- D507 pad 1: GND -> /frontend_temp/GND
- D508 pad 2: GND -> /frontend_temp/GND
- D509 pad 1: GND -> /frontend_temp/GND
- D510 pad 2: GND -> /frontend_temp/GND
- D511 pad 1: GND -> /frontend_temp/GND
- D512 pad 2: GND -> /frontend_temp/GND
- D513 pad 1: GND -> /frontend_temp/GND
- D702 pad 1: GND -> /frontend_bridge/GND
- D702 pad 4: GND -> /frontend_bridge/GND
- D703 pad 1: GND -> /frontend_bridge/GND
- D703 pad 4: GND -> /frontend_bridge/GND
- D704 pad 1: GND -> /frontend_bridge/GND
- D704 pad 4: GND -> /frontend_bridge/GND
- D705 pad 2: GND -> /frontend_bridge/GND
- D706 pad 1: GND -> /frontend_bridge/GND
- D707 pad 2: GND -> /frontend_bridge/GND
- D708 pad 1: GND -> /frontend_bridge/GND
- D802 pad 3: GND -> /CAN/GND
- H101 pad 1: (no net) -> Earth
- H102 pad 1: (no net) -> Earth
- H103 pad 1: (no net) -> Earth
- H104 pad 1: (no net) -> Earth
- H105 pad 1: (no net) -> Earth
- H106 pad 1: (no net) -> Earth
- J102 pad 2: GND -> /Power/V+
- J107 pad 1: /Digital Output/OUT0 -> /Digital Output/OUT4
- J107 pad 2: /Digital Output/OUT1 -> /Digital Output/OUT5
- J107 pad 3: /Digital Output/OUT2 -> /Digital Output/OUT6
- J107 pad 4: /Digital Output/OUT3 -> /Digital Output/OUT7
- J108 pad 1: /Digital Output/OUT4 -> /frontend_420/4200
- J108 pad 2: /Digital Output/OUT5 -> /frontend_420/4201
- J108 pad 3: /Digital Output/OUT6 -> /frontend_420/4202
- J108 pad 4: /Digital Output/OUT7 -> /frontend_420/4203
- J109 pad 1: /frontend_420/4200 -> /frontend_bridge/B0_5V+
- J109 pad 2: /frontend_420/4201 -> /frontend_bridge/B0+
- J109 pad 3: /frontend_420/4202 -> /frontend_bridge/B0-
- J109 pad 4: /frontend_420/4203 -> /frontend_bridge/B0_GND
- J110 pad 1: /frontend_bridge/B0_5V+ -> /frontend_bridge/B1_5V+
- J110 pad 2: /frontend_bridge/B0+ -> /frontend_bridge/B1+
- J110 pad 3: /frontend_bridge/B0- -> /frontend_bridge/B1-
- J110 pad 4: /frontend_bridge/B0_GND -> /frontend_bridge/B1_GND
- J111 pad 1: /frontend_bridge/B1_5V+ -> /frontend_temp/TC0+
- J111 pad 2: /frontend_bridge/B1+ -> /frontend_temp/TC0-
- J111 pad 3: /frontend_bridge/B1- -> /frontend_temp/TC1+
- J111 pad 4: /frontend_bridge/B1_GND -> /frontend_temp/TC1-
- J112 pad 1: /frontend_temp/TC0+ -> /frontend_temp/TC2+
- J112 pad 2: /frontend_temp/TC0- -> /frontend_temp/TC2-
- J112 pad 3: /frontend_temp/TC1+ -> /frontend_temp/TC3+
- J112 pad 4: /frontend_temp/TC1- -> /frontend_temp/TC3-
- L1101 pad 8: +24V -> /Power/FlyBuck/+24V_PRIM
- R1102 pad 2: +POE -> /Power/CDB
- R1106 pad 1: Earth -> /Power/FlyBuck/+24V_PRIM
- R1106 pad 2: GND -> /Power/FlyBuck/FB
- R1107 pad 1: +24V -> /Power/FlyBuck/FB
- R1107 pad 2: /Power/FlyBuck/FB -> /Power/GND_ISO
- R1108 pad 1: /Power/FlyBuck/FB -> /Power/FlyBuck/SW
- R1108 pad 2: /Power/GND_ISO -> /Power/FlyBuck/A
- R213 pad 1: Earth -> Net-(C208-Pad2)
- R213 pad 2: GND -> Earth
- R214 pad 1: Net-(C208-Pad2) -> Net-(C209-Pad2)
- R215 pad 1: Net-(C209-Pad2) -> Net-(C210-Pad2)
- R216 pad 1: Net-(C210-Pad2) -> Net-(C211-Pad2)
- R217 pad 1: Net-(C211-Pad2) -> /Ethernet/LED1
- R217 pad 2: Earth -> Net-(J201-Pad11)
- R218 pad 1: /Ethernet/LED1 -> /Ethernet/LED2
- R218 pad 2: Net-(J201-Pad11) -> Net-(J201-Pad9)
- R408 pad 1: Net-(U403-~{MR}) -> Net-(R408-Pad1)
- R408 pad 2: +3.3V -> /MCU/~{QSPI_SS}
- R409 pad 1: Net-(R409-Pad1) -> +3.3V
- R409 pad 2: /MCU/~{QSPI_SS} -> Net-(U402-~{CS})
- R410 pad 1: +3.3V -> Net-(U402-~{CS})
- R410 pad 2: Net-(U402-~{CS}) -> /MCU/~{QSPI_SS}
- R411 pad 1: Net-(U402-~{CS}) -> /MCU/USB_D-
- R411 pad 2: /MCU/~{QSPI_SS} -> Net-(U403-USB_DP)
- R412 pad 1: /EN -> Net-(C415-Pad2)
- R412 pad 2: /MCU/~{RST} -> Net-(U403-XOUT)
- R413 pad 1: /MCU/USB_D- -> /MCU/~{RST}
- R413 pad 2: Net-(U404-USB_DP) -> +3.3V
- R414 pad 1: Net-(C416-Pad2) -> /MCU/USB_D+
- R414 pad 2: Net-(U404-XOUT) -> Net-(U403-USB_DM)
- R415 pad 1: /MCU/~{RST} -> /MCU/I2C0.SDA
- R416 pad 1: /MCU/USB_D+ -> /MCU/I2C0.SCL
- R416 pad 2: Net-(U404-USB_DM) -> +3.3V
- R417 pad 1: /MCU/I2C0.SDA -> /MCU/I2C1.SDA
- R418 pad 1: /MCU/I2C0.SCL -> /MCU/I2C1.SCL
- R419 pad 1: /MCU/I2C1.SDA -> /MCU/I2C2.SDA
- R420 pad 1: /MCU/I2C1.SCL -> /MCU/I2C2.SCL
- R421 pad 1: /MCU/I2C2.SDA -> Net-(U404-~{MR})
- R422 pad 1: /MCU/I2C2.SCL -> +3.3V
- R422 pad 2: +3.3V -> Net-(U404-V_{DD})
- R501 pad 2: +3.3V -> /frontend_temp/+3.3V
- R502 pad 2: +3.3V -> /frontend_temp/+3.3V
- R503 pad 1: +3.3V -> /frontend_temp/+3.3V
- R504 pad 2: +3.3V -> /frontend_temp/+3.3V
- R505 pad 2: +3.3V -> /frontend_temp/+3.3V
- R506 pad 1: GND -> /frontend_temp/GND
- R507 pad 2: +3.3V -> /frontend_temp/+3.3V
- R508 pad 2: +3.3V -> /frontend_temp/+3.3V
- R509 pad 1: GND -> /frontend_temp/GND
- R510 pad 1: +3.3V -> /frontend_temp/+3.3V
- R519 pad 2: +3.3V -> /frontend_temp/+3.3V
- R520 pad 1: GND -> /frontend_temp/GND
- R521 pad 2: +3.3V -> /frontend_temp/+3.3V
- R522 pad 1: GND -> /frontend_temp/GND
- R523 pad 2: +3.3V -> /frontend_temp/+3.3V
- R524 pad 1: GND -> /frontend_temp/GND
- R525 pad 2: +3.3V -> /frontend_temp/+3.3V
- R526 pad 1: GND -> /frontend_temp/GND
- R705 pad 1: GND -> /frontend_bridge/GND
- R706 pad 1: GND -> /frontend_bridge/GND
- R712 pad 1: GND -> /frontend_bridge/GND
- R714 pad 1: GND -> /frontend_bridge/GND
- R717 pad 2: GND -> /frontend_bridge/GND
- R718 pad 2: GND -> /frontend_bridge/GND
- R803 pad 2: GND -> /CAN/GND
- TP401 pad 1: Net-(R409-Pad1) -> Net-(R408-Pad1)
- TR201 pad 1: /Ethernet/TXP -> /Ethernet/RXN
- TR201 pad 10: /Ethernet/POE-36 -> /Ethernet/POE+12
- TR201 pad 11: /Ethernet/RX_P -> /Ethernet/TX_N
- TR201 pad 14: /Ethernet/TX_N -> /Ethernet/RX_P
- TR201 pad 15: /Ethernet/POE+12 -> /Ethernet/POE-36
- TR201 pad 16: /Ethernet/TX_P -> /Ethernet/RX_N
- TR201 pad 3: /Ethernet/TXN -> /Ethernet/RXP
- TR201 pad 6: /Ethernet/RXP -> /Ethernet/TXN
- TR201 pad 8: /Ethernet/RXN -> /Ethernet/TXP
- TR201 pad 9: /Ethernet/RX_N -> /Ethernet/TX_P
- U1102 pad 3: +24V -> /Power/FlyBuck/+24V_PRIM
- U401 pad 11: unconnected-(U401-P07-Pad11) -> /MCU/WDI
- U401 pad 20: /MCU/WDI -> unconnected-(U401-P17-Pad20)
- U403 pad 1: /MCU/~{RST} -> +3.3V
- U403 pad 2: GND -> /MCU/I2C0.SDA
- U403 pad 3: Net-(U403-~{MR}) -> /MCU/I2C0.SCL
- U403 pad 4: /MCU/WDI -> /MCU/SPI0.SCK
- U403 pad 5: +3.3V -> /MCU/SPI0.TX
- U404 pad 1: +3.3V -> /MCU/~{RST}
- U404 pad 2: /MCU/I2C0.SDA -> GND
- U404 pad 3: /MCU/I2C0.SCL -> Net-(U404-~{MR})
- U404 pad 4: /MCU/SPI0.SCK -> /MCU/WDI
- U404 pad 5: /MCU/SPI0.TX -> Net-(U404-V_{DD})
- U501 pad 3: GND -> /frontend_temp/GND
- U502 pad 5: GND -> /frontend_temp/GND
- U502 pad 8: +3.3V -> /frontend_temp/+3.3V
- U503 pad 5: GND -> /frontend_temp/GND
- U503 pad 8: +3.3V -> /frontend_temp/+3.3V
- U504 pad 2: GND -> /frontend_temp/GND
- U504 pad 5: +3.3V -> /frontend_temp/+3.3V
- U505 pad 1: GND -> /frontend_temp/GND
- U505 pad 2: +3.3V -> /frontend_temp/+3.3V
- U506 pad 2: GND -> /frontend_temp/GND
- U506 pad 5: +3.3V -> /frontend_temp/+3.3V
- U507 pad 3: GND -> /frontend_temp/GND
- U507 pad 8: +3.3V -> /frontend_temp/+3.3V
- U508 pad 3: GND -> /frontend_temp/GND
- U508 pad 8: +3.3V -> /frontend_temp/+3.3V
- U701 pad 1: GND_ISO -> GND
- U701 pad 2: +5V_ISO -> +5V
- U701 pad 3: GND -> /frontend_bridge/GND
- U702 pad 15: GND -> /frontend_bridge/GND
- U702 pad 9: GND -> /frontend_bridge/GND
- U703 pad 15: GND -> /frontend_bridge/GND
- U703 pad 9: GND -> /frontend_bridge/GND
- U704 pad 4: GND -> /frontend_bridge/GND
- U704 pad 5: GND -> /frontend_bridge/GND
- U705 pad 4: GND -> /frontend_bridge/GND
- U705 pad 5: GND -> /frontend_bridge/GND
- U801 pad 1: GND_ISO -> GND
- U801 pad 2: +5V_ISO -> +5V
- U801 pad 3: GND -> /CAN/GND
- U802 pad 7: GND -> /CAN/GND
- Y401 pad 1: Net-(U404-XIN) -> Net-(U403-XIN)
- Y401 pad 3: Net-(C416-Pad2) -> Net-(C415-Pad2)
Other:
- board size 160 x 70 mm -> 160 x 68 mm

Commit message: inital placement done
Parts:
- removed C1202: 10uF, Capacitor_SMD:C_0805_2012Metric
- removed R1003, R1004, R1303, R1304, R501, R502, R601, R602: 1k, Resistor_SMD:R_0402_1005Metric
- removed R803: 0, Resistor_SMD:R_0402_1005Metric
- removed U1201: ER_OLEDM0.91_1x-I2C, Display:ER_OLEDM0.91_1x-I2C
- added C527: 10uF, Capacitor_SMD:C_0805_2012Metric, B.Cu at (208.7, 80.2)
- added D709: BAV199DW, Package_TO_SOT_SMD:SOT-363_SC-70-6, F.Cu at (176.5, 99.5)
- C103, C301, C401, C403, C404, C405, C406, C407, C408, C413, C414, C415, C501, C502, C504, C505, C508, C510, C511, C512, C513, C515, C516, C517, C518, C519, C520, C521, C522, C523, C524, C525, C526, C601, C602, C603, C604, C605, C606, C607, C608, C701, C703, C704, C706, C714, C715, C716, C717, C718, C719, C801, C802, C803, C903, C904, C905, C906, C909, C910, C911, C912, D506, D507, D508, D509, D510, D511, D512, D513, D603, D604, D605, D606, D705, D706, D707, D708, D801, F701, F702, FB501, FB701, FB801, J401, Q702, R1009, R1012, R102, R1023, R1024, R1025, R1026, R1027, R1028, R1029, R1030, R217, R218, R401, R402, R403, R404, R408, R409, R410, R411, R412, R414, R415, R416, R507, R508, R511, R512, R513, R514, R515, R516, R517, R518, R519, R520, R521, R522, R523, R524, R525, R526, R527, R603, R604, R605, R606, R702, R704, R705, R706, R707, R708, R709, R710, R711, R712, R713, R714, R717, R718, R719, R802, R903, R904, R905, R906, R907, R908, R909, R910, R913, R914, R915, R916, R917, R918, R919, R920, TP401, TP402, TP403, U1001, U1002, U1003, U401, U404, U502, U505, U703, U704, U705, U803, U901, U902, U903, U904: moved to B.Cu
- J402: footprint Connector_PinHeader_2.54mm:PinHeader_1x03_P2.54mm_Vertical_SMD_Pin1Left -> Connector_PinHeader_2.54mm:PinHeader_1x03_P2.54mm_Vertical
- moved FID101 269.2 mm to (62.0, 86.0)
- moved R801 266.7 mm to (70.0, 128.0), turned to 180 degrees
- moved U803 256.0 mm to (74.5, 127.5)
- moved U802 254.3 mm to (74.5, 126.0)
- moved D802 253.9 mm to (80.5, 127.5)
- moved FB801 252.6 mm to (81.0, 118.0)
- moved C802 251.6 mm to (71.0, 123.0), turned to 180 degrees
- moved R802 250.6 mm to (84.5, 123.0)
- moved C801 249.6 mm to (72.5, 117.5), turned to 90 degrees
- moved D801 248.4 mm to (79.0, 123.5)
- moved R218 247.9 mm to (75.3, 64.5), turned to 90 degrees
- moved R217 246.2 mm to (77.0, 64.5), turned to 90 degrees
- moved C803 243.8 mm to (77.5, 118.0), turned to 180 degrees
- moved C804 241.2 mm to (79.5, 124.5), turned to -90 degrees
- moved C805 240.8 mm to (81.0, 124.0), turned to -90 degrees
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Connections:
- C504 pad 1: unconnected-(C504-Pad1) -> Net-(U501-+Vout)
- C803 pad 2: /CAN/GND -> /CAN/CAN_GND
- C804 pad 2: /CAN/GND -> /CAN/CAN_GND
- C805 pad 2: /CAN/GND -> /CAN/CAN_GND
- D702 pad 3: /frontend_bridge/+5V_SENSE0 -> (no net)
- D702 pad 4: /frontend_bridge/GND -> (no net)
- D702 pad 5: /frontend_bridge/+5V -> (no net)
- D802 pad 3: /CAN/GND -> /CAN/CAN_GND
- J101 pad 1: /CAN/CAN_H -> /CAN/CAN_L
- J101 pad 2: /CAN/CAN_L -> /CAN/CAN_H
- J103 pad 1: /Power Output/OUT0 -> /Power Output/OUT1
- J103 pad 2: /Power Output/OUT1 -> /Power Output/OUT0
- R507 pad 1: /MCU/I2C0.SCL -> /frontend_temp/SCL
- R508 pad 1: /MCU/I2C0.SDA -> /frontend_temp/SDA
- U1301 pad 3: Net-(U1301-IN3) -> unconnected-(U1301-IN3-Pad3)
- U1301 pad 4: Net-(U1301-IN4) -> unconnected-(U1301-IN4-Pad4)
- U1301 pad 7: /FAULT_PWR -> unconnected-(U1301-~{ST3}-Pad7)
- U1301 pad 8: /FAULT_PWR -> unconnected-(U1301-~{ST4}-Pad8)
- U502 pad 6: /MCU/I2C0.SCL -> /frontend_temp/SCL
- U502 pad 7: /MCU/I2C0.SDA -> /frontend_temp/SDA
- U504 pad 7: /frontend_temp/TC2- -> /frontend_temp/TC3-
- U507 pad 10: /MCU/I2C0.SCL -> /frontend_temp/SCL
- U507 pad 9: /MCU/I2C0.SDA -> /frontend_temp/SDA
- U508 pad 10: /MCU/I2C0.SCL -> /frontend_temp/SCL
- U508 pad 9: /MCU/I2C0.SDA -> /frontend_temp/SDA
- U801 pad 3: /CAN/GND -> /CAN/CAN_GND
- U802 pad 7: /CAN/GND -> /CAN/CAN_GND
Routing:
- net Net-(U403-USB_DP): track 0.00 -> 5.98 mm, vias 0 -> 1
- net Net-(U403-USB_DM): track 0.00 -> 4.65 mm, vias 0 -> 1
