File: hardware/c0-dev/indicators.kicad_sch (KiCad schematic)
At the start: 6 parts

Commit message: silkscreen, isolation and placement cleanup
Parts:
- D1201, D1202, D1203, D1204: footprint LED_SMD:LED_WS2812B_PLCC4_5.0x5.0mm_P3.2mm -> conduit:LED_WS2812B-Mini_PLCC4_3.5x3.5mm
